Commit message: URDF: J2/J3 limits 2.5 deg inside the robot hard limits (I-term pushed J3 to 140.1)

File: igus_rebel_description_real/urdf/igus_rebel.urdf (robot description, URDF)
Before this commit: robot igus_rebel, 12 links, 11 joints
Joints:
- joint joint2: limit lower=-1.3800 upper=2.4435 effort=330 velocity=2.16 -> lower=-1.3500 upper=2.4435 effort=330 velocity=2.16
- joint joint3: limit lower=-1.39626 upper=2.4300 effort=330 velocity=2.16 -> lower=-1.39626 upper=2.4000 effort=330 velocity=2.16
